Commit message: Update 112 files
- /egu_50_description/CMakeLists.txt
- /egu_50_description/config/joint_names_egu_50_fingers_08_16.yaml
- /egu_50_description/doc/.gitkeep
- /egu_50_description/doc/EGU_50_misaligned.jpg
- /egu_50_description/doc/EGU_50_version_1.png
- /egu_50_description/doc/EGU_50_version_2.png
- /egu_50_description/launch/display.launch
- /egu_50_description/launch/egu_50.launch
- /egu_50_description/launch/load_egu_50.launch
- /egu_50_description/meshes/base_link.dae
- /egu_50_description/meshes/finger_link_left.STL
- /egu_50_description/meshes/finger_link_right.STL
- /egu_50_description/meshes/fingers_base_link_left.STL
- /egu_50_description/meshes/fingers_base_link_right.STL
- /egu_50_description/meshes/gripper_base_link_left.dae
- /egu_50_description/meshes/gripper_base_link_right.dae
- /egu_50_description/meshes/gripper_finger_down.dae
- /egu_50_description/meshes/gripper_finger_up.dae
- /egu_50_description/meshes/screw_1.STL
- /egu_50_description/meshes/screw_1.dae
- /egu_50_description/meshes/screw_2.STL
- /egu_50_description/meshes/screw_2.dae
- /egu_50_description/meshes/screw_3.STL
- /egu_50_description/meshes/screw_3.dae
- /egu_50_description/meshes/screw_4.STL
- /egu_50_description/meshes/screw_4.dae
- /egu_50_description/meshes/symbol_1_left.dae
- /egu_50_description/meshes/symbol_1_right.dae
- /egu_50_description/meshes/symbol_2_left.STL
- /egu_50_description/meshes/symbol_2_left.dae
- /egu_50_description/meshes/symbol_2_right.STL
- /egu_50_description/meshes/symbol_2_right.dae
- /egu_50_description/meshes/translational_left.dae
- /egu_50_description/meshes/translational_right.dae
- /egu_50_description/package.xml
- /egu_50_description/readme.md
- /egu_50_description/urdf/egu_50.gazebo.xacro
- /egu_50_description/urdf/egu_50.transmission.xacro
- /egu_50_description/urdf/egu_50.urdf.xacro
- /egu_50_description/urdf/egu_50.xacro
- /egu_50_description/urdf/egu_50_base_link.urdf.xacro
- /egu_50_description/urdf/egu_50_base_link.xacro
- /egu_50_description/urdf/egu_50_fingers_link.urdf.xacro
- /egu_50_description/urdf/egu_50_fingers_link.xacro
- /egu_50_description/urdf/egu_50_fingers_version2_link.urdf.xacro
- /egu_50_description/urdf/egu_50_fingers_version2_link.xacro
- /egu_50_ur_description/CMakeLists.txt
- /egu_50_ur_description/doc/.gitkeep
- /egu_50_ur_description/doc/EGU_50_and_UR_10e.png
- /egu_50_ur_description/launch/load_ur_egu.launch
- /egu_50_ur_description/package.xml
- /egu_50_ur_description/readme.md
- /egu_50_ur_description/urdf/ur_egu.urdf.xacro
- /egu_50_ur_description/urdf/ur_egu.xacro
- /egu_description/config/joint_names_egu_50_fingers_08_16.yaml
- /egu_description/doc/.gitkeep
- /egu_description/doc/EGU_50_version_1.png
- /egu_description/doc/EGU_50_version_2.png
- /egu_description/doc/EGU_50_misaligned.jpg
- /egu_description/launch/display.launch
- /egu_description/launch/egu_50.launch
- /egu_description/launch/load_egu_50.launch
- /egu_description/meshes/fingers_base_link_left.STL
- /egu_description/meshes/finger_link_left.STL
- /egu_description/meshes/fingers_base_link_right.STL
- /egu_description/meshes/finger_link_right.STL
- /egu_description/meshes/gripper_finger_down.dae
- /egu_description/meshes/screw_3.STL
- /egu_description/meshes/gripper_finger_up.dae
- /egu_description/meshes/gripper_base_link_left.dae
- /egu_description/meshes/screw_1.dae
- /egu_description/meshes/gripper_base_link_right.dae
- /egu_description/meshes/base_link.dae
- /egu_description/meshes/screw_1.STL
- /egu_description/meshes/screw_2.dae
- /egu_description/meshes/screw_2.STL
- /egu_description/meshes/symbol_1_right.dae
- /egu_description/meshes/screw_4.STL
- /egu_description/meshes/screw_4.dae
- /egu_description/meshes/screw_3.dae
- /egu_description/meshes/symbol_1_left.dae
- /egu_description/meshes/symbol_2_right.STL
- /egu_description/meshes/translational_left.dae
- /egu_description/meshes/symbol_2_left.dae
- /egu_description/meshes/symbol_2_right.dae
- /egu_description/meshes/translational_right.dae
- /egu_description/meshes/symbol_2_left.STL
- /egu_description/urdf/egu_50_base_link.xacro
- /egu_description/urdf/egu_50_base_link.urdf.xacro
- /egu_description/urdf/egu_50_fingers_link.urdf.xacro
- /egu_description/urdf/egu_50_fingers_link.xacro
- /egu_description/urdf/egu_50_fingers_version2_link.urdf.xacro
- /egu_description/urdf/egu_50_fingers_version2_link.xacro
- /egu_description/urdf/egu_50.gazebo.xacro
- /egu_description/urdf/egu_50.transmission.xacro
- /egu_description/urdf/egu_50.transmission.urdf.xacro
- /egu_description/urdf/egu_50.urdf.xacro
- /egu_description/urdf/egu_50.xacro
- /egu_description/CMakeLists.txt
- /egu_description/package.xml
- /egu_description/readme.md
- /ur_schunk_gripper_description/doc/.gitkeep
- /ur_schunk_gripper_description/doc/EGU_50_and_UR_10e.png
- /ur_schunk_gripper_description/launch/display.launch
- /ur_schunk_gripper_description/launch/load_ur_schunk_gripper.launch
- /ur_schunk_gripper_description/launch/gazebo.launch
- /ur_schunk_gripper_description/urdf/ur_schunk_gripper.urdf.xacro
- /ur_schunk_gripper_description/urdf/ur_schunk_gripper.xacro
- /ur_schunk_gripper_description/readme.md
- /ur_schunk_gripper_description/config/robot_model.rviz
- /ur_schunk_gripper_description/CMakeLists.txt
- /ur_schunk_gripper_description/package.xml

File: egu_description/urdf/egu_50.xacro (robot description, xacro)
@@ -4,12 +4,13 @@
     <xacro:macro name="egu_50" params="prefix_1 prefix_2 meshType">
         <!-- imports -->
-        <xacro:include filename="$(find egu_50_description)/urdf/egu_50_base_link.urdf.xacro" />
-        <xacro:include filename="$(find egu_50_description)/urdf/egu_50_fingers_link.urdf.xacro" />
-        <xacro:include filename="$(find egu_50_description)/urdf/egu_50_fingers_version2_link.urdf.xacro" />
-        <!--xacro:include filename="$(find egu_50_description)/urdf/egu_50.gazebo.xacro" /-->
-        <xacro:include filename="$(find egu_50_description)/urdf/egu_50.transmission.xacro" />
+        <xacro:include filename="$(find egu_description)/urdf/egu_50_base_link.urdf.xacro" />
+        <xacro:include filename="$(find egu_description)/urdf/egu_50_fingers_link.urdf.xacro" />
+        <xacro:include filename="$(find egu_description)/urdf/egu_50_fingers_version2_link.urdf.xacro" />
+        <!--xacro:include filename="$(find egu_description)/urdf/egu_50.gazebo.xacro" /-->
+        <xacro:include filename="$(find egu_description)/urdf/egu_50.transmission.xacro" />
         <xacro:egu_50_base_link prefix="${prefix_1}_" meshType="${meshType}" />
         <!--xacro:egu_50_fingers_link prefix="${prefix_2}_" meshType="${meshType}" /-->
-        <xacro:egu_50_fingers_version2_link prefix="${prefix_2}_" meshType="STL" />
+        <xacro:egu_50_fingers_link prefix="${prefix_2}_" meshType="${meshType}" />
+        <xacro:egu_50_transmission prefix="${prefix_2}_" />
         <!-- links -->
         <!--link name="world" /-->
@@ -20,5 +21,5 @@
         </joint>
 -->
-        <joint name="fixed_joint_gripper_base_link_right" type="fixed">
+        <!-- <joint name="fixed_joint_gripper_base_link_right" type="fixed">
           <origin xyz="0.018 0 0.01" rpy="1.5708 0 -1.5708" />
           <parent link="${prefix_1}_translational_right" />
@@ -31,6 +32,5 @@
           <child link="${prefix_2}_base_link_left" />
           <axis xyz="0 0 0" />
-        </joint>
-<!--
+        </joint> -->
         <joint name="fixed_joint_gripper_base_link_right" type="fixed">
           <origin xyz="0.018 0 0.01" rpy="0 0 0" />
@@ -45,5 +45,4 @@
           <axis xyz="0 0 0" />
         </joint>
--->
     </xacro:macro>
 </robot>

File: egu_description/urdf/egu_50_base_link.urdf.xacro (robot description, xacro)
@@ -1,5 +1,5 @@
 <?xml version="1.0"?>
 <robot name="egu_50_base_link" xmlns:xacro="http://www.ros.org/wiki/xacro">
-   <xacro:include filename="$(find egu_50_description)/urdf/egu_50_base_link.xacro" />
+   <xacro:include filename="$(find egu_description)/urdf/egu_50_base_link.xacro" />
    <!-- xacro:egu_50_base_link prefix="" meshType="dae" / -->
 </robot>

File: egu_description/urdf/egu_50_base_link.xacro (robot description, xacro)
@@ -28,5 +28,5 @@
         <geometry>
           <mesh
-            filename="package://egu_50_description/meshes/base_link.${meshType}" />
+            filename="package://egu_description/meshes/base_link.${meshType}" />
         </geometry>
         <material name="light_blue_1" />
@@ -38,5 +38,5 @@
         <geometry>
           <mesh
-            filename="package://egu_50_description/meshes/base_link.${meshType}" />
+            filename="package://egu_description/meshes/base_link.${meshType}" />
         </geometry>
       </collision>
@@ -63,5 +63,5 @@
         <geometry>
           <mesh
-            filename="package://egu_50_description/meshes/symbol_1_left.${meshType}" />
+            filename="package://egu_description/meshes/symbol_1_left.${meshType}" />
         </geometry>
         <material name="light_blue_1" />
@@ -73,5 +73,5 @@
         <geometry>
           <mesh
-            filename="package://egu_50_description/meshes/symbol_1_left.${meshType}" />
+            filename="package://egu_description/meshes/symbol_1_left.${meshType}" />
         </geometry>
       </collision>
@@ -98,5 +98,5 @@
         <geometry>
           <mesh
-            filename="package://egu_50_description/meshes/symbol_1_right.${meshType}" />
+            filename="package://egu_description/meshes/symbol_1_right.${meshType}" />
         </geometry>
         <material name="light_blue_1" />
@@ -108,5 +108,5 @@
         <geometry>
           <mesh
-            filename="package://egu_50_description/meshes/symbol_1_right.${meshType}" />
+            filename="package://egu_description/meshes/symbol_1_right.${meshType}" />
         </geometry>
       </collision>
@@ -134,5 +134,5 @@
         <geometry>
           <mesh
-            filename="package://egu_50_description/meshes/translational_left.${meshType}" />
+            filename="package://egu_description/meshes/translational_left.${meshType}" />
         </geometry>
         <material name="light_grey" />
@@ -144,5 +144,5 @@
         <geometry>
           <mesh
-            filename="package://egu_50_description/meshes/translational_left.${meshType}" />
+            filename="package://egu_description/meshes/translational_left.${meshType}" />
         </geometry>
       </collision>
@@ -170,5 +170,5 @@
         <geometry>
           <mesh
-            filename="package://egu_50_description/meshes/translational_right.${meshType}" />
+            filename="package://egu_description/meshes/translational_right.${meshType}" />
         </geometry>
         <material name="light_grey" />
@@ -180,5 +180,5 @@
         <geometry>
           <mesh
-            filename="package://egu_50_description/meshes/translational_right.${meshType}" />
+            filename="package://egu_description/meshes/translational_right.${meshType}" />
         </geometry>
       </collision>
@@ -212,5 +212,5 @@
     </joint>
     <joint
-      name="${prefix}prismatic_joint_translational_left"
+      name="${prefix}prismatic_1"
       type="prismatic">
       <origin
@@ -231,5 +231,5 @@
     </joint>
     <joint
-      name="${prefix}prismatic_joint_translational_right"
+      name="${prefix}prismatic_2"
       type="prismatic">
       <origin
@@ -247,5 +247,5 @@
         effort="300"
         velocity="0.11" />
-      <mimic joint="${prefix}prismatic_joint_translational_left" multiplier="-1" offset="0" />
+      <mimic joint="${prefix}prismatic_1" multiplier="-1" offset="0" />
       <dynamics damping="0.3" friction="0.2" />
     </joint>

File: egu_description/urdf/egu_50_fingers_link.urdf.xacro (robot description, xacro)
@@ -1,5 +1,5 @@
 <?xml version="1.0"?>
 <robot name="egu_50_fingers_link" xmlns:xacro="http://www.ros.org/wiki/xacro">
-   <xacro:include filename="$(find egu_50_description)/urdf/egu_50_fingers_link.xacro" />
+   <xacro:include filename="$(find egu_description)/urdf/egu_50_fingers_link.xacro" />
    <!-- xacro:egu_50_fingers_link prefix="" meshType="dae" / -->
 </robot>

File: egu_description/urdf/egu_50_fingers_link.xacro (robot description, xacro)
@@ -19,12 +19,12 @@
         <origin xyz="0 0 0" rpy="0 0 0" />
         <geometry>
-          <mesh filename="package://egu_50_description/meshes/gripper_base_link_left.${meshType}" />
-        </geometry>
-        <material name="light_blue" />
-      </visual>
-      <collision>
-        <origin xyz="0 0 0" rpy="0 0 0" />
-        <geometry>
-          <mesh filename="package://egu_50_description/meshes/gripper_base_link_left.${meshType}" />
+          <mesh filename="package://egu_description/meshes/gripper_base_link_left.${meshType}" />
+        </geometry>
+        <material name="light_blue" />
+      </visual>
+      <collision>
+        <origin xyz="0 0 0" rpy="0 0 0" />
+        <geometry>
+          <mesh filename="package://egu_description/meshes/gripper_base_link_left.${meshType}" />
         </geometry>
       </collision>
@@ -39,12 +39,12 @@
         <origin xyz="0 0 0" rpy="0 0 0" />
         <geometry>
-          <mesh filename="package://egu_50_description/meshes/gripper_base_link_right.${meshType}" />
-        </geometry>
-        <material name="light_blue" />
-      </visual>
-      <collision>
-        <origin xyz="0 0 0" rpy="0 0 0" />
-        <geometry>
-          <mesh filename="package://egu_50_description/meshes/gripper_base_link_right.${meshType}" />
+          <mesh filename="package://egu_description/meshes/gripper_base_link_right.${meshType}" />
+        </geometry>
+        <material name="light_blue" />
+      </visual>
+      <collision>
+        <origin xyz="0 0 0" rpy="0 0 0" />
+        <geometry>
+          <mesh filename="package://egu_description/meshes/gripper_base_link_right.${meshType}" />
         </geometry>
       </collision>
@@ -59,12 +59,12 @@
         <origin xyz="0 0 0" rpy="0 0 0" />
         <geometry>
-          <mesh filename="package://egu_50_description/meshes/gripper_finger_down.${meshType}" />
-        </geometry>
-        <material name="light_blue" />
-      </visual>
-      <collision>
-        <origin xyz="0 0 0" rpy="0 0 0" />
-        <geometry>
-          <mesh filename="package://egu_50_description/meshes/gripper_finger_down.${meshType}" />
+          <mesh filename="package://egu_description/meshes/gripper_finger_down.${meshType}" />
+        </geometry>
+        <material name="light_blue" />
+      </visual>
+      <collision>
+        <origin xyz="0 0 0" rpy="0 0 0" />
+        <geometry>
+          <mesh filename="package://egu_description/meshes/gripper_finger_down.${meshType}" />
         </geometry>
       </collision>
@@ -79,12 +79,12 @@
         <origin xyz="0 0 0" rpy="0 0 0" />
         <geometry>
-          <mesh filename="package://egu_50_description/meshes/gripper_finger_up.${meshType}" />
-        </geometry>
-        <material name="light_blue" />
-      </visual>
-      <collision>
-        <origin xyz="0 0 0" rpy="0 0 0" />
-        <geometry>
-          <mesh filename="package://egu_50_description/meshes/gripper_finger_up.${meshType}" />
+          <mesh filename="package://egu_description/meshes/gripper_finger_up.${meshType}" />
+        </geometry>
+        <material name="light_blue" />
+      </visual>
+      <collision>
+        <origin xyz="0 0 0" rpy="0 0 0" />
+        <geometry>
+          <mesh filename="package://egu_description/meshes/gripper_finger_up.${meshType}" />
         </geometry>
       </collision>
@@ -99,12 +99,12 @@
         <origin xyz="0 0 0" rpy="0 0 0" />
         <geometry>
-          <mesh filename="package://egu_50_description/meshes/symbol_2_left.${meshType}" />
-        </geometry>
-        <material name="light_blue" />
-      </visual>
-      <collision>
-        <origin xyz="0 0 0" rpy="0 0 0" />
-        <geometry>
-          <mesh filename="package://egu_50_description/meshes/symbol_2_left.${meshType}" />
+          <mesh filename="package://egu_description/meshes/symbol_2_left.${meshType}" />
+        </geometry>
+        <material name="light_blue" />
+      </visual>
+      <collision>
+        <origin xyz="0 0 0" rpy="0 0 0" />
+        <geometry>
+          <mesh filename="package://egu_description/meshes/symbol_2_left.${meshType}" />
         </geometry>
       </collision>
@@ -119,12 +119,12 @@
         <origin xyz="0 0 0" rpy="0 0 0" />
         <geometry>
-          <mesh filename="package://egu_50_description/meshes/symbol_2_right.${meshType}" />
-        </geometry>
-        <material name="light_blue" />
-      </visual>
-      <collision>
-        <origin xyz="0 0 0" rpy="0 0 0" />
-        <geometry>
-          <mesh filename="package://egu_50_description/meshes/symbol_2_right.${meshType}" />
+          <mesh filename="package://egu_description/meshes/symbol_2_right.${meshType}" />
+        </geometry>
+        <material name="light_blue" />
+      </visual>
+      <collision>
+        <origin xyz="0 0 0" rpy="0 0 0" />
+        <geometry>
+          <mesh filename="package://egu_description/meshes/symbol_2_right.${meshType}" />
         </geometry>
       </collision>
@@ -139,5 +139,5 @@
         <origin xyz="0 0 0" rpy="0 0 0" />
         <geometry>
-          <mesh filename="package://egu_50_description/meshes/screw_1.${meshType}" />
+          <mesh filename="package://egu_description/meshes/screw_1.${meshType}" />
         </geometry>
         <material name="grey" />
@@ -146,5 +146,5 @@
         <origin xyz="0 0 0" rpy="0 0 0" />
         <geometry>
-          <mesh filename="package://egu_50_description/meshes/screw_1.${meshType}" />
+          <mesh filename="package://egu_description/meshes/screw_1.${meshType}" />
         </geometry>
       </collision>
@@ -158,5 +158,5 @@
       <visual>
         <origin xyz="0 0 0" rpy="0 0 0" />
-        <geometry> <mesh filename="package://egu_50_description/meshes/screw_2.${meshType}" />
+        <geometry> <mesh filename="package://egu_description/meshes/screw_2.${meshType}" />
         </geometry>
         <material name="grey" />
@@ -165,5 +165,5 @@
         <origin xyz="0 0 0" rpy="0 0 0" />
         <geometry>
-          <mesh filename="package://egu_50_description/meshes/screw_2.${meshType}" />
+          <mesh filename="package://egu_description/meshes/screw_2.${meshType}" />
         </geometry>
       </collision>
@@ -178,5 +178,5 @@
         <origin xyz="0 0 0" rpy="0 0 0" />
         <geometry>
-          <mesh filename="package://egu_50_description/meshes/screw_3.${meshType}" />
+          <mesh filename="package://egu_description/meshes/screw_3.${meshType}" />
         </geometry>
         <material name="grey" />
@@ -185,5 +185,5 @@
         <origin xyz="0 0 0" rpy="0 0 0" />
         <geometry>
-          <mesh filename="package://egu_50_description/meshes/screw_3.${meshType}" />
+          <mesh filename="package://egu_description/meshes/screw_3.${meshType}" />
         </geometry>
       </collision>
@@ -198,5 +198,5 @@
         <origin xyz="0 0 0" rpy="0 0 0" />
         <geometry>
-          <mesh filename="package://egu_50_description/meshes/screw_4.${meshType}" />
+          <mesh filename="package://egu_description/meshes/screw_4.${meshType}" />
         </geometry>
         <material name="grey" />
@@ -205,5 +205,5 @@
         <origin xyz="0 0 0" rpy="0 0 0" />
         <geometry>
-          <mesh filename="package://egu_50_description/meshes/screw_4.${meshType}" />
+          <mesh filename="package://egu_description/meshes/screw_4.${meshType}" />
         </geometry>
       </collision>

File: egu_description/urdf/egu_50_fingers_version2_link.urdf.xacro (robot description, xacro)
@@ -1,5 +1,5 @@
 <?xml version="1.0"?>
 <robot name="egu_50_fingers_version2_link" xmlns:xacro="http://www.ros.org/wiki/xacro">
-   <xacro:include filename="$(find egu_50_description)/urdf/egu_50_fingers_version2_link.xacro" />
+   <xacro:include filename="$(find egu_description)/urdf/egu_50_fingers_version2_link.xacro" />
    <!-- xacro:egu_50_fingers_link prefix="" meshType="dae" / -->
 </robot>
