Commit message: Update 112 files
- /egu_50_description/CMakeLists.txt
- /egu_50_description/config/joint_names_egu_50_fingers_08_16.yaml
- /egu_50_description/doc/.gitkeep
- /egu_50_description/doc/EGU_50_misaligned.jpg
- /egu_50_description/doc/EGU_50_version_1.png
- /egu_50_description/doc/EGU_50_version_2.png
- /egu_50_description/launch/display.launch
- /egu_50_description/launch/egu_50.launch
- /egu_50_description/launch/load_egu_50.launch
- /egu_50_description/meshes/base_link.dae
- /egu_50_description/meshes/finger_link_left.STL
- /egu_50_description/meshes/finger_link_right.STL
- /egu_50_description/meshes/fingers_base_link_left.STL
- /egu_50_description/meshes/fingers_base_link_right.STL
- /egu_50_description/meshes/gripper_base_link_left.dae
- /egu_50_description/meshes/gripper_base_link_right.dae
- /egu_50_description/meshes/gripper_finger_down.dae
- /egu_50_description/meshes/gripper_finger_up.dae
- /egu_50_description/meshes/screw_1.STL
- /egu_50_description/meshes/screw_1.dae
- /egu_50_description/meshes/screw_2.STL
- /egu_50_description/meshes/screw_2.dae
- /egu_50_description/meshes/screw_3.STL
- /egu_50_description/meshes/screw_3.dae
- /egu_50_description/meshes/screw_4.STL
- /egu_50_description/meshes/screw_4.dae
- /egu_50_description/meshes/symbol_1_left.dae
- /egu_50_description/meshes/symbol_1_right.dae
- /egu_50_description/meshes/symbol_2_left.STL
- /egu_50_description/meshes/symbol_2_left.dae
- /egu_50_description/meshes/symbol_2_right.STL
- /egu_50_description/meshes/symbol_2_right.dae
- /egu_50_description/meshes/translational_left.dae
- /egu_50_description/meshes/translational_right.dae
- /egu_50_description/package.xml
- /egu_50_description/readme.md
- /egu_50_description/urdf/egu_50.gazebo.xacro
- /egu_50_description/urdf/egu_50.transmission.xacro
- /egu_50_description/urdf/egu_50.urdf.xacro
- /egu_50_description/urdf/egu_50.xacro
- /egu_50_description/urdf/egu_50_base_link.urdf.xacro
- /egu_50_description/urdf/egu_50_base_link.xacro
- /egu_50_description/urdf/egu_50_fingers_link.urdf.xacro
- /egu_50_description/urdf/egu_50_fingers_link.xacro
- /egu_50_description/urdf/egu_50_fingers_version2_link.urdf.xacro
- /egu_50_description/urdf/egu_50_fingers_version2_link.xacro
- /egu_50_ur_description/CMakeLists.txt
- /egu_50_ur_description/doc/.gitkeep
- /egu_50_ur_description/doc/EGU_50_and_UR_10e.png
- /egu_50_ur_description/launch/load_ur_egu.launch
- /egu_50_ur_description/package.xml
- /egu_50_ur_description/readme.md
- /egu_50_ur_description/urdf/ur_egu.urdf.xacro
- /egu_50_ur_description/urdf/ur_egu.xacro
- /egu_description/config/joint_names_egu_50_fingers_08_16.yaml
- /egu_description/doc/.gitkeep
- /egu_description/doc/EGU_50_version_1.png
- /egu_description/doc/EGU_50_version_2.png
- /egu_description/doc/EGU_50_misaligned.jpg
- /egu_description/launch/display.launch
- /egu_description/launch/egu_50.launch
- /egu_description/launch/load_egu_50.launch
- /egu_description/meshes/fingers_base_link_left.STL
- /egu_description/meshes/finger_link_left.STL
- /egu_description/meshes/fingers_base_link_right.STL
- /egu_description/meshes/finger_link_right.STL
- /egu_description/meshes/gripper_finger_down.dae
- /egu_description/meshes/screw_3.STL
- /egu_description/meshes/gripper_finger_up.dae
- /egu_description/meshes/gripper_base_link_left.dae
- /egu_description/meshes/screw_1.dae
- /egu_description/meshes/gripper_base_link_right.dae
- /egu_description/meshes/base_link.dae
- /egu_description/meshes/screw_1.STL
- /egu_description/meshes/screw_2.dae
- /egu_description/meshes/screw_2.STL
- /egu_description/meshes/symbol_1_right.dae
- /egu_description/meshes/screw_4.STL
- /egu_description/meshes/screw_4.dae
- /egu_description/meshes/screw_3.dae
- /egu_description/meshes/symbol_1_left.dae
- /egu_description/meshes/symbol_2_right.STL
- /egu_description/meshes/translational_left.dae
- /egu_description/meshes/symbol_2_left.dae
- /egu_description/meshes/symbol_2_right.dae
- /egu_description/meshes/translational_right.dae
- /egu_description/meshes/symbol_2_left.STL
- /egu_description/urdf/egu_50_base_link.xacro
- /egu_description/urdf/egu_50_base_link.urdf.xacro
- /egu_description/urdf/egu_50_fingers_link.urdf.xacro
- /egu_description/urdf/egu_50_fingers_link.xacro
- /egu_description/urdf/egu_50_fingers_version2_link.urdf.xacro
- /egu_description/urdf/egu_50_fingers_version2_link.xacro
- /egu_description/urdf/egu_50.gazebo.xacro
- /egu_description/urdf/egu_50.transmission.xacro
- /egu_description/urdf/egu_50.transmission.urdf.xacro
- /egu_description/urdf/egu_50.urdf.xacro
- /egu_description/urdf/egu_50.xacro
- /egu_description/CMakeLists.txt
- /egu_description/package.xml
- /egu_description/readme.md
- /ur_schunk_gripper_description/doc/.gitkeep
- /ur_schunk_gripper_description/doc/EGU_50_and_UR_10e.png
- /ur_schunk_gripper_description/launch/display.launch
- /ur_schunk_gripper_description/launch/load_ur_schunk_gripper.launch
- /ur_schunk_gripper_description/launch/gazebo.launch
- /ur_schunk_gripper_description/urdf/ur_schunk_gripper.urdf.xacro
- /ur_schunk_gripper_description/urdf/ur_schunk_gripper.xacro
- /ur_schunk_gripper_description/readme.md
- /ur_schunk_gripper_description/config/robot_model.rviz
- /ur_schunk_gripper_description/CMakeLists.txt
- /ur_schunk_gripper_description/package.xml

File: egu_description/urdf/egu_50_fingers_version2_link.xacro (robot description, xacro)
@@ -24,5 +24,5 @@
       <geometry>
         <mesh
-          filename="package://egu_50_description/meshes/fingers_base_link_left.${meshType}" />
+          filename="package://egu_description/meshes/fingers_base_link_left.${meshType}" />
       </geometry>
       <material
@@ -38,5 +38,5 @@
       <geometry>
         <mesh
-          filename="package://egu_50_description/meshes/fingers_base_link_left.${meshType}" />
+          filename="package://egu_description/meshes/fingers_base_link_left.${meshType}" />
       </geometry>
     </collision>
@@ -64,5 +64,5 @@
       <geometry>
         <mesh
-          filename="package://egu_50_description/meshes/finger_link_left.${meshType}" />
+          filename="package://egu_description/meshes/finger_link_left.${meshType}" />
       </geometry>
       <material
@@ -78,5 +78,5 @@
       <geometry>
         <mesh
-          filename="package://egu_50_description/meshes/finger_link_left.${meshType}" />
+          filename="package://egu_description/meshes/finger_link_left.${meshType}" />
       </geometry>
     </collision>
@@ -104,5 +104,5 @@
       <geometry>
         <mesh
-          filename="package://egu_50_description/meshes/fingers_base_link_right.${meshType}" />
+          filename="package://egu_description/meshes/fingers_base_link_right.${meshType}" />
       </geometry>
       <material
@@ -118,5 +118,5 @@
       <geometry>
         <mesh
-          filename="package://egu_50_description/meshes/fingers_base_link_right.${meshType}" />
+          filename="package://egu_description/meshes/fingers_base_link_right.${meshType}" />
       </geometry>
     </collision>
@@ -144,5 +144,5 @@
       <geometry>
         <mesh
-          filename="package://egu_50_description/meshes/finger_link_right.${meshType}" />
+          filename="package://egu_description/meshes/finger_link_right.${meshType}" />
       </geometry>
       <material
@@ -158,5 +158,5 @@
       <geometry>
         <mesh
-          filename="package://egu_50_description/meshes/finger_link_right.${meshType}" />
+          filename="package://egu_description/meshes/finger_link_right.${meshType}" />
       </geometry>
     </collision>
@@ -184,5 +184,5 @@
       <geometry>
         <mesh
-          filename="package://egu_50_description/meshes/screw_1.${meshType}" />
+          filename="package://egu_description/meshes/screw_1.${meshType}" />
       </geometry>
       <material
@@ -198,5 +198,5 @@
       <geometry>
         <mesh
-          filename="package://egu_50_description/meshes/screw_1.${meshType}" />
+          filename="package://egu_description/meshes/screw_1.${meshType}" />
       </geometry>
     </collision>
@@ -224,5 +224,5 @@
       <geometry>
         <mesh
-          filename="package://egu_50_description/meshes/screw_2.${meshType}" />
+          filename="package://egu_description/meshes/screw_2.${meshType}" />
       </geometry>
       <material
@@ -238,5 +238,5 @@
       <geometry>
         <mesh
-          filename="package://egu_50_description/meshes/screw_2.${meshType}" />
+          filename="package://egu_description/meshes/screw_2.${meshType}" />
       </geometry>
     </collision>
@@ -264,5 +264,5 @@
       <geometry>
         <mesh
-          filename="package://egu_50_description/meshes/screw_3.${meshType}" />
+          filename="package://egu_description/meshes/screw_3.${meshType}" />
       </geometry>
       <material
@@ -278,5 +278,5 @@
       <geometry>
         <mesh
-          filename="package://egu_50_description/meshes/screw_3.${meshType}" />
+          filename="package://egu_description/meshes/screw_3.${meshType}" />
       </geometry>
     </collision>
@@ -304,5 +304,5 @@
       <geometry>
         <mesh
-          filename="package://egu_50_description/meshes/screw_4.${meshType}" />
+          filename="package://egu_description/meshes/screw_4.${meshType}" />
       </geometry>
       <material
@@ -318,5 +318,5 @@
       <geometry>
         <mesh
-          filename="package://egu_50_description/meshes/screw_4.${meshType}" />
+          filename="package://egu_description/meshes/screw_4.${meshType}" />
       </geometry>
     </collision>
@@ -344,5 +344,5 @@
       <geometry>
         <mesh
-          filename="package://egu_50_description/meshes/symbol_2_left.${meshType}" />
+          filename="package://egu_description/meshes/symbol_2_left.${meshType}" />
       </geometry>
       <material
@@ -358,5 +358,5 @@
       <geometry>
         <mesh
-          filename="package://egu_50_description/meshes/symbol_2_left.${meshType}" />
+          filename="package://egu_description/meshes/symbol_2_left.${meshType}" />
       </geometry>
     </collision>
@@ -384,5 +384,5 @@
       <geometry>
         <mesh
-          filename="package://egu_50_description/meshes/symbol_2_right.${meshType}" />
+          filename="package://egu_description/meshes/symbol_2_right.${meshType}" />
       </geometry>
       <material
@@ -398,5 +398,5 @@
       <geometry>
         <mesh
-          filename="package://egu_50_description/meshes/symbol_2_right.${meshType}" />
+          filename="package://egu_description/meshes/symbol_2_right.${meshType}" />
       </geometry>
     </collision>
@@ -509,14 +509,12 @@
     <kp>1000000.0</kp>
     <kd>1.0</kd>
-    <mu1>1.0</mu1>
-    <mu2>1.0</mu2>
-    <minDepth>0.001</minDepth>
+    <mu>0.35</mu>
+    <mu2>0.35</mu2>
   </gazebo>
   <gazebo reference="${prefix}finger_right">
     <kp>1000000.0</kp>
     <kd>1.0</kd>
-    <mu1>1.0</mu1>
-    <mu2>1.0</mu2>
-    <minDepth>0.001</minDepth>
+    <mu>0.35</mu>
+    <mu2>0.35</mu2>
   </gazebo>
  </xacro:macro>
