Commit message: Update 2 files
- /ur_schunk_gripper_description/urdf/ur_schunk_gripper.xacro
- /ur_schunk_gripper_description/urdf/ur_schunk_gripper.urdf.xacro

File: ur_schunk_gripper_description/urdf/ur_schunk_gripper.urdf.xacro (robot description, xacro)
@@ -1,7 +1,18 @@
 <?xml version="1.0"?>
 <robot xmlns:xacro="http://wiki.ros.org/xacro" name="ur_schunk_gripper_robot">
+  <!-- Existing parameters -->
   <xacro:arg name="ur_model" default="ur10e"/>
   <xacro:arg name="gripper_type" default="pzv"/>
+  <!-- New parameters with their default values -->
+  <xacro:arg name="world_joint_xyz" default="0 0 0"/>
+  <xacro:arg name="world_joint_rpy" default="0 0 0"/>
+  <!-- Include the xacro file that contains the macro definition -->
   <xacro:include filename="$(find ur_schunk_gripper_description)/urdf/ur_schunk_gripper.xacro"/>
-  <xacro:ur_schunk_gripper_robot ur_model="$(arg ur_model)" gripper_type="$(arg gripper_type)"/>
+  <!-- Call the macro with all parameters, including the new ones -->
+  <xacro:ur_schunk_gripper_robot
+    ur_model="$(arg ur_model)"
+    gripper_type="$(arg gripper_type)"
+    world_joint_xyz="$(arg world_joint_xyz)"
+    world_joint_rpy="$(arg world_joint_rpy)"
+  />
 </robot>

File: ur_schunk_gripper_description/urdf/ur_schunk_gripper.xacro (robot description, xacro)
@@ -9,4 +9,6 @@
    safety_k_position:=20
    gripper_type
+   world_joint_xyz:='0 0 0'
+   world_joint_rpy:='0 0 0'
    ">
     <xacro:property name="joint_limits_parameters_file" value="$(find ur_description)/config/${ur_model}/joint_limits.yaml"/>
@@ -78,5 +80,5 @@
       <parent link="world"/>1
       <child link="base_link"/>
-      <origin xyz="0 0 0" rpy="0 0 0"/>
+      <origin xyz="${world_joint_xyz}" rpy="${world_joint_rpy}"/>
     </joint>
     <link name="tool0_controller"/>
